File: Schematics/Cap RTC-MCP79400.kicad_pcb (KiCad board)
At the start: 2 copper layers, 49.5 x 30.5 mm, 15 parts, among them K1 CAP_CONN_LHS, K2 CAP_CONN_RHS, U1 MCP7400, X1 32.768 kHz

Commit message: Cosmetic Changes to Silkscreen
Cosmetic Changes to Silkscreen
Parts:
- added REF**: Symbol_OSHW-Logo_SilkScreen, Toadstool:Symbol_OSHW-Logo_SilkScreen, F.Cu at (226.1, 108.0)
Other:
- board text added: "v1.0 2015-08-06"
- board text removed: "v0.1 2015-04-18"

Commit message: Silkscreen changes
Added label to MFP pin
New Gerber files generated
Other:
- board text added: "MFP"
